Commit message: minor changes to fit project

File: husky_description/urdf/accessories/vlp16_mount.urdf.xacro (robot description, xacro)
@@ -56,5 +56,5 @@
       <origin xyz="0 -0.04 ${height/2}" rpy="0 0 0"/>
     </joint>
-    <xacro:VLP-16 parent="${prefix}vlp16_mount_base_link" topic="${topic}">
+    <xacro:VLP-16 parent="${prefix}vlp16_mount_base_link" topic="${topic}" gpu="true">
       <origin xyz="0 0 ${height}" rpy="0 0 0" />
     </xacro:VLP-16>

File: husky_description/urdf/husky.urdf.xacro (robot description, xacro)
@@ -23,5 +23,4 @@
 <robot name="husky" xmlns:xacro="http://ros.org/wiki/xacro">
   <xacro:arg name="laser_enabled" default="$(optenv HUSKY_LMS1XX_ENABLED 0)" />
-  <!--xacro:arg name="laser_xyz" default="$(optenv HUSKY_LMS1XX_XYZ 0.2206 0.0 0.00635)" /-->
   <xacro:arg name="laser_xyz" default="$(optenv HUSKY_LMS1XX_XYZ -0.3 0.0 0.6)" />
   <xacro:arg name="laser_rpy" default="$(optenv HUSKY_LMS1XX_RPY 0.0 0.0 0.0)" />
@@ -30,16 +29,10 @@
   <xacro:arg name="laser_secondary_rpy" default="$(optenv HUSKY_LMS1XX_SECONDARY_RPY 0.0 0.0 3.14159)" />
   <xacro:arg name="laser_3d_enabled" default="$(optenv HUSKY_LASER_3D_ENABLED 0)" />
-  <xacro:arg name="laser_3d_xyz" default="$(optenv HUSKY_LASER_3D_XYZ 0 0 0)" />
+  <xacro:arg name="laser_3d_xyz" default="$(optenv HUSKY_LASER_3D_XYZ -0.3 0.0 0.6)" />
   <xacro:arg name="laser_3d_rpy" default="$(optenv HUSKY_LASER_3D_RPY 0 0 0)" />
   <xacro:arg name="realsense_enabled" default="$(optenv HUSKY_REALSENSE_ENABLED 0)" />
-  <xacro:arg name="realsense2_enabled" default="$(optenv HUSKY_REALSENSE2_ENABLED 0)" />
-  <!-- CAMERA TO ARM ATTACHMENT: Changed position, rotation and parent mount point -->
-  <xacro:arg name="realsense_xyz" default="$(optenv HUSKY_REALSENSE_XYZ 0.0 0.08 0.05)" />
+  <xacro:arg name="realsense_xyz" default="$(optenv HUSKY_REALSENSE_XYZ 0.0 0.08 1)" />
   <xacro:arg name="realsense_rpy" default="$(optenv HUSKY_REALSENSE_RPY 0 0 1.5707963)" />
   <xacro:arg name="realsense_mount" default="$(optenv HUSKY_REALSENSE_MOUNT_FRAME ur_arm_wrist_2_link)" />
-  <!-- SETUP FOR SECOND REALSENSE CAMERA-->
-  <xacro:arg name="realsense2_xyz" default="$(optenv HUSKY_REALSENSE_XYZ 0.0 0.0 0.1)" />
-  <xacro:arg name="realsense2_rpy" default="$(optenv HUSKY_REALSENSE_RPY 0 0 0)" />
-  <xacro:arg name="realsense2_mount" default="$(optenv HUSKY_REALSENSE_MOUNT_FRAME front_bumper_link)" />
   <xacro:property name="husky_front_bumper_extend" value="$(optenv HUSKY_FRONT_BUMPER_EXTEND 0)" />
   <xacro:property name="husky_rear_bumper_extend" value="$(optenv HUSKY_REAR_BUMPER_EXTEND 0)" />
@@ -53,5 +46,4 @@
   <xacro:include filename="$(find husky_description)/urdf/wheel.urdf.xacro" />
   <xacro:include filename="$(find husky_description)/urdf/accessories/intel_realsense.urdf.xacro"/>
-  <xacro:include filename="$(find husky_description)/urdf/accessories/intel_realsense2.urdf.xacro"/> <!-- include 2nd Realsense file-->
   <xacro:include filename="$(find husky_description)/urdf/accessories/sick_lms1xx_mount.urdf.xacro"/>
   <xacro:include filename="$(find husky_description)/urdf/accessories/sensor_arch.urdf.xacro"/>
@@ -177,18 +169,9 @@
     <xacro:intel_realsense_mount prefix="camera" topic="realsense" parent_link="realsense_mountpoint"/>
   </xacro:if>
-  <xacro:if value="$(arg realsense2_enabled)">
-    <link name="realsense2_mountpoint"/>
-    <joint name="realsense2_mountpoint_joint" type="fixed">
-      <origin xyz="$(arg realsense2_xyz)" rpy="$(arg realsense2_rpy)" />
-      <parent link="$(arg realsense2_mount)"/>
-      <child link="realsense2_mountpoint" />
-    </joint>
-    <xacro:intel_realsense2_mount prefix="camera2" topic="realsense2" parent_link="realsense2_mountpoint"/>
-  </xacro:if>
   <!--
     Add the 3d laser to the sensor arch if needed
   -->
   <xacro:if value="$(arg laser_3d_enabled)">
-    <xacro:vlp16_mount prefix="" parent_link="sensor_arch_mount_link" topic="$(optenv HUSKY_LASER_3D_TOPIC points)">
+    <xacro:vlp16_mount prefix="vlp16" parent_link="top_plate_link" topic="$(optenv HUSKY_LASER_3D_TOPIC /vlp16/points)">
       <origin xyz="$(arg laser_3d_xyz)" rpy="$(arg laser_3d_rpy)" />
     </xacro:vlp16_mount>
